File: EEG_ADS1299.sch (KiCad schematic (older format))
At the start: 70 parts, among them IC1 ADS1299, P1 CONN_2, P2 CONN_2, P3 CONN_1, P4 CONN_1, P5 CONN_01X06, U1 TPS61221, U2 TPS61222, U3 NRF528XX-QFAA, U4 MPU-9250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

Commit message: Updated schematic, deleted extra pin headers. Removed extra components from pcb file.
Parts:
- removed P3, P4: CONN_1, Pin_Headers:Pin_Header_Straight_1x01_Pitch2.54mm, symbol CONN_1
- renumbered P5 to P3
Connections:
- net labels removed: SRB1
- wire segments 312 -> 310
Changed lines of the file:
@@
 Text GLabel 12900 9850 0    60   Input ~ 0
 AVDD
-Text Label 4250 7700 2    60   ~ 0
-SRB1
 Text GLabel 29100 4700 3    60   Input ~ 0
 DGND
@@
 	1    0    0    -1
 $EndComp
-Text Label 4300 7350 2    60   ~ 0
-BIASIN
 Text Label 23500 6300 1    60   ~ 0
 DOUT
@@
 $EndComp
 NoConn ~ 14550 12000
-$Comp
-L CONN_1 P4
-U 1 1 58B800EE
-P 3400 7350
-F 0 "P4" V 3350 7350 40  0000 C CNN
-F 1 "CONN_1" V 3450 7350 40  0000 C CNN
-F 2 "Pin_Headers:Pin_Header_Straight_1x01_Pitch2.54mm" H 3400 7350 60  0001 C CNN
-F 3 "" H 3400 7350 60  0000 C CNN
-	1    3400 7350
-	-1   0    0    1
-$EndComp
 Text GLabel 13650 3750 0    60   Input ~ 0
 AVSS
@@
 IN1-
 $Comp
-L CONN_1 P3
-U 1 1 591A6E5B
-P 3400 7700
-F 0 "P3" V 3350 7700 40  0000 C CNN
-F 1 "CONN_1" V 3450 7700 40  0000 C CNN
-F 2 "Pin_Headers:Pin_Header_Straight_1x01_Pitch2.54mm" H 3400 7700 60  0001 C CNN
-F 3 "" H 3400 7700 60  0000 C CNN
-	1    3400 7700
-	-1   0    0    1
-$EndComp
-$Comp
 L NRF528XX-QFAA-RESCUE-EEG_ADS1299_2 U3
 U 1 1 597FEAA6
@@
 	13800 6350 13800 6600
 Wire Wire Line
-	3750 7350 4300 7350
-Wire Wire Line
 	15150 12250 15350 12250
 Wire Wire Line
@@
 	500  6100 5350 6100
 Wire Wire Line
-	3750 7700 4250 7700
-Wire Wire Line
 	2450 7000 2450 7150
 Wire Wire Line
@@
 Connection ~ 9900 11650
 $Comp
-L CONN_01X06 P5
+L CONN_01X06 P3
 U 1 1 5A2786C7
 P 8800 10900
-F 0 "P5" H 8800 11250 50  0000 C CNN
+F 0 "P3" H 8800 11250 50  0000 C CNN
 F 1 "CONN_01X06" V 8900 10900 50  0000 C CNN
 F 2 "Pin_Headers:Pin_Header_Straight_1x06_Pitch2.54mm" H 8800 10900 50  0001 C CNN

Commit message: Finished pcb draft for 4-ch with 2x INA828 (single-ended only).
Parts:
- U5, U6: footprint Housings_SOIC:HTSOP-8-1EP_3.9x4.9mm_Pitch1.27mm -> INA828:SOIC_8_4.9mm_x_3.91
Changed lines of the file:
@@
 LIBS:texas_TPS61222
 LIBS:EEG_ADS1299_2-cache
+LIBS:EEG_ADS1299-cache
 EELAYER 25 0
 EELAYER END
@@
 F 0 "U5" H 10750 10575 50  0000 L CNN
 F 1 "INA828" H 10750 10325 50  0000 L CNN
-F 2 "Housings_SOIC:HTSOP-8-1EP_3.9x4.9mm_Pitch1.27mm" H 10700 10450 50  0001 C CNN
+F 2 "INA828:SOIC_8_4.9mm_x_3.91" H 10700 10450 50  0001 C CNN
 F 3 "" H 10700 10450 50  0001 C CNN
 	1    10600 10450
@@
 F 0 "U6" H 10750 11575 50  0000 L CNN
 F 1 "INA828" H 10750 11325 50  0000 L CNN
-F 2 "Housings_SOIC:HTSOP-8-1EP_3.9x4.9mm_Pitch1.27mm" H 10700 11450 50  0001 C CNN
+F 2 "INA828:SOIC_8_4.9mm_x_3.91" H 10700 11450 50  0001 C CNN
 F 3 "" H 10700 11450 50  0001 C CNN
 	1    10600 11450
