File: EEG_ADS1299.kicad_pcb (KiCad board)
At the start: 2 copper layers, 48.5 x 21.7 mm, 76 parts, among them IC1 ADS1299, P1 CONN_2, P2 CONN_2, P3 CONN_01X08, U1 TPS2294x, U2 TPS61222, U3 NRF528XX-QFAA, U4 MPU-9250, U5 INA828, U6 INA828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

Commit message: Updated schematic and pcb design to reflect final EEG design: Connected SRB1 to IN12-.
Connections:
- IC1 pad 17: Net-(IC1-Pad17) -> /IN12-
- P3 pad 1: /IN1 -> /REF_ELECTRODE
- P3 pad 3: /IN2 -> /REF_ELECTRODE
- U5 pad 3: /IN2 -> /REF_ELECTRODE
- U6 pad 3: /IN1 -> /REF_ELECTRODE
Routing:
- net /REF_ELECTRODE: track 0.00 -> 18.8 mm
- net /IN2: track 6.33 -> 0.00 mm
- net /IN12-: track 9.95 -> 16.1 mm, vias 0 -> 2
- net /IN1: track 5.68 -> 0.00 mm
